File: Loaf/PCB/PLC_Input_Slice/_restore_backup_2026-09-25T09-14-27-361/BREAD_slice_v2.kicad_sch (KiCad schematic)
At the start: 26 parts, among them J1 10018783-10200TLF, J3 DB25_Socket, U1 MCP4922-EP, U2 MCP4922-EP, U3 MCP4922-EP, U4 MCP4922-EP, U5 MCP3208, U6 MCP2561-E-P, U7 MCP2515-xSO, Y1 16MHZ Crystal

Commit message: Preliminary PCB Design
Parts:
- removed R3, R4, R5, R6: 10k, R_Axial_DIN0207_L6.3mm_D2.5mm_P10.16mm_Horizontal, symbol Device:R_US
- added C1: C, Package_SO:SOIC-8_3.9x4.9mm_P1.27mm, symbol Device:C
- Y2: renamed from Y1; footprint Crystal_HC49-4H_Vertical -> LOAF Update:XTAL_ECS-160-20-3X-TR
- renumbered C1 to C5, C2 to C7, R2 to R15, R1 to R16
Connections:
- net +5V: no longer J3.20 (P20), J3.7
- net AIO0: now also J3.1, RN1.9 (R8), U4.14 (VoutA); no longer J3.13, RN2.2 (R1), U1.10 (VoutB)
- net AIO1: now also J3.14 (P14), RN1.8 (R7), U4.10 (VoutB); no longer J3.25 (P25), RN2.3 (R2), U1.14 (VoutA)
- net AIO2: now also J3.2, RN1.7 (R6), U3.14 (VoutA); no longer J3.12, RN2.4 (R3), U2.10 (VoutB)
- net AIO3: now also J3.15 (P15), RN1.6 (R5), U3.10 (VoutB); no longer J3.24 (P24), RN2.5 (R4), U2.14 (VoutA)
- net AIO4: now also J3.3, RN1.5 (R4), U2.14 (VoutA); no longer J3.11, RN2.6 (R5), U3.10 (VoutB)
- net AIO5: now also J3.16 (P16), RN1.4 (R3), U2.10 (VoutB); no longer J3.23 (P23), RN2.7 (R6), U3.14 (VoutA)
- net AIO6: now also J3.4, RN1.3 (R2), U1.14 (VoutA); no longer J3.10, RN2.8 (R7), U4.10 (VoutB)
- net AIO7: now also J3.17 (P17), RN1.2 (R1), U1.10 (VoutB); no longer J3.22 (P22), RN2.9 (R8), U4.14 (VoutA)
- net DIO0: now also J3.13, RN2.2 (R1); no longer J3.1, RN1.9 (R8)
- net DIO1: now also J3.25 (P25), RN2.3 (R2); no longer J3.14 (P14), RN1.8 (R7)
- net DIO2: now also J3.12, RN2.4 (R3); no longer J3.2, RN1.7 (R6)
- net DIO3: now also J3.24 (P24), RN2.5 (R4); no longer J3.15 (P15), RN1.6 (R5)
- net DIO4: now also J3.11, RN2.6 (R5); no longer J3.3, RN1.5 (R4)
- net DIO5: now also J3.23 (P23), RN2.7 (R6); no longer J3.16 (P16), RN1.4 (R3)
- net DIO6: now also J3.10, RN2.8 (R7); no longer J3.4, RN1.3 (R2)
- net DIO7: now also J3.22 (P22), RN2.9 (R8); no longer J3.17 (P17), RN1.2 (R1)
- net GND: now also J3.18 (P18), J3.19 (P19), J3.20 (P20), J3.5, J3.6, J3.7
- net ESTOP: no longer names the net of A1.20 (A1)
- net ESTOP: no longer J3.6
- net RESET: no longer names the net of A1.28 (~{RESET})
- net RESET: no longer J3.19 (P19)
- net SHDNTRIG: no longer names the net of A1.19 (A0)
- net URX: no longer names the net of A1.2 (RX1)
- net URX: no longer J3.18 (P18)
- net UTX: no longer names the net of A1.1 (TX1)
- net UTX: no longer J3.5
- no-connect marks 20 -> 18
