File: Loaf/PCB/PLC_Input_Slice/BREAD_slice_v2.kicad_pcb (KiCad board)
At the start: 2 copper layers, 100 x 70.6 mm, 31 parts, among them J1 10018783-10200TLF, J2 Barrel_Jack, J3 DB25_Socket, U1 MCP4922-EP, U2 MCP4922-EP, U3 MCP4922-EP, U4 MCP4922-EP, U5 MCP3208, U6 MCP2561-E-P, U7 MCP2515-xSO, Y1 16MHZ Crystal

Commit message: Updated Daughter Board
Parts:
- U5: footprint Package_DIP:DIP-16_W7.62mm_LongPads -> Package_DIP:DIP-16_W7.62mm
Changed lines of the file:
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@@
 		)
 	)
-	(footprint "Package_DIP:DIP-16_W7.62mm_LongPads"
+	(footprint "Package_DIP:DIP-16_W7.62mm"
 		(layer "F.Cu")
 		(at 190.627 70.95 -90)
-		(descr "16-lead though-hole mounted DIP package, row spacing 7.62mm (300 mils), LongPads")
-		(tags "THT DIP DIL PDIP 2.54mm 7.62mm 300mil LongPads")
+		(descr "16-lead though-hole mounted DIP package, row spacing 7.62mm (300 mils)")
+		(tags "THT DIP DIL PDIP 2.54mm 7.62mm 300mil")
 		(property "Reference" "U5"
 			(at 3.81 -2.33 90)
@@
 		(duplicate_pad_numbers_are_jumpers no)
 		(fp_line
-			(start 1.56 19.11)
-			(end 6.06 19.11)
+			(start 1.16 19.11)
+			(end 6.46 19.11)
 			(stroke
 				(width 0.12)
@@
 		)
 		(fp_line
-			(start 6.06 19.11)
-			(end 6.06 -1.33)
+			(start 6.46 19.11)
+			(end 6.46 -1.33)
 			(stroke
 				(width 0.12)
@@
 		)
 		(fp_line
-			(start 1.56 -1.33)
-			(end 1.56 19.11)
+			(start 1.16 -1.33)
+			(end 1.16 19.11)
 			(stroke
 				(width 0.12)
@@
 		(fp_line
 			(start 2.81 -1.33)
-			(end 1.56 -1.33)
+			(end 1.16 -1.33)
 			(stroke
 				(width 0.12)
@@
 		)
 		(fp_line
-			(start 6.06 -1.33)
+			(start 6.46 -1.33)
 			(end 4.81 -1.33)
 			(stroke
@@
 		)
 		(fp_rect
-			(start -1.45 -1.52)
-			(end 9.07 19.3)
+			(start -1.06 -1.52)
+			(end 8.67 19.3)
 			(stroke
 				(width 0.05)
@@
 		(pad "1" thru_hole roundrect
 			(at 0 0 270)
-			(size 2.4 1.6)
+			(size 1.6 1.6)
 			(drill 0.8)
 			(layers "*.Cu" "*.Mask")
@@
 			(pintype "input")
 		)
-		(pad "2" thru_hole oval
+		(pad "2" thru_hole circle
 			(at 0 2.54 270)
-			(size 2.4 1.6)
+			(size 1.6 1.6)
 			(drill 0.8)
 			(layers "*.Cu" "*.Mask")
@@
 			(pintype "input")
 		)
-		(pad "3" thru_hole oval
+		(pad "3" thru_hole circle
 			(at 0 5.08 270)
-			(size 2.4 1.6)
+			(size 1.6 1.6)
 			(drill 0.8)
 			(layers "*.Cu" "*.Mask")
@@
 			(pintype "input")
 		)
-		(pad "4" thru_hole oval
+		(pad "4" thru_hole circle
 			(at 0 7.62 270)
-			(size 2.4 1.6)
+			(size 1.6 1.6)
 			(drill 0.8)
 			(layers "*.Cu" "*.Mask")
@@
 			(pintype "input")
 		)
-		(pad "5" thru_hole oval
+		(pad "5" thru_hole circle
 			(at 0 10.16 270)
-			(size 2.4 1.6)
+			(size 1.6 1.6)
 			(drill 0.8)
 			(layers "*.Cu" "*.Mask")
@@
 			(pintype "input")
 		)
-		(pad "6" thru_hole oval
+		(pad "6" thru_hole circle
 			(at 0 12.7 270)
-			(size 2.4 1.6)
+			(size 1.6 1.6)
 			(drill 0.8)
 			(layers "*.Cu" "*.Mask")
@@
 			(pintype "input")
 		)
-		(pad "7" thru_hole oval
+		(pad "7" thru_hole circle
 			(at 0 15.24 270)
-			(size 2.4 1.6)
+			(size 1.6 1.6)
 			(drill 0.8)
 			(layers "*.Cu" "*.Mask")
@@
 			(pintype "input")
 		)
-		(pad "8" thru_hole oval
+		(pad "8" thru_hole circle
 			(at 0 17.78 270)
-			(size 2.4 1.6)
+			(size 1.6 1.6)
 			(drill 0.8)
 			(layers "*.Cu" "*.Mask")
@@
 			(pintype "input")
 		)
-		(pad "9" thru_hole oval
+		(pad "9" thru_hole circle
 			(at 7.62 17.78 270)
-			(size 2.4 1.6)
+			(size 1.6 1.6)
 			(drill 0.8)
 			(layers "*.Cu" "*.Mask")
@@
 			(pintype "power_in")
 		)
-		(pad "10" thru_hole oval
+		(pad "10" thru_hole circle
 			(at 7.62 15.24 270)
-			(size 2.4 1.6)
+			(size 1.6 1.6)
 			(drill 0.8)
 			(layers "*.Cu" "*.Mask")
@@
 			(pintype "input")
 		)
-		(pad "11" thru_hole oval
+		(pad "11" thru_hole circle
 			(at 7.62 12.7 270)
-			(size 2.4 1.6)
+			(size 1.6 1.6)
 			(drill 0.8)
 			(layers "*.Cu" "*.Mask")
@@
 			(pintype "input")
 		)
-		(pad "12" thru_hole oval
+		(pad "12" thru_hole circle
 			(at 7.62 10.16 270)
-			(size 2.4 1.6)
+			(size 1.6 1.6)
 			(drill 0.8)
 			(layers "*.Cu" "*.Mask")
@@
 			(pintype "output")
 		)
-		(pad "13" thru_hole oval
+		(pad "13" thru_hole circle
 			(at 7.62 7.62 270)
-			(size 2.4 1.6)
+			(size 1.6 1.6)
 			(drill 0.8)
 			(layers "*.Cu" "*.Mask")
@@
 			(pintype "input")
 		)
-		(pad "14" thru_hole oval
+		(pad "14" thru_hole circle
 			(at 7.62 5.08 270)
-			(size 2.4 1.6)
+			(size 1.6 1.6)
 			(drill 0.8)
 			(layers "*.Cu" "*.Mask")
@@
 			(pintype "power_in")
 		)
-		(pad "15" thru_hole oval
+		(pad "15" thru_hole circle
 			(at 7.62 2.54 270)
-			(size 2.4 1.6)
+			(size 1.6 1.6)
 			(drill 0.8)
 			(layers "*.Cu" "*.Mask")
@@
 			(pintype "power_in")
 		)
-		(pad "16" thru_hole oval
+		(pad "16" thru_hole circle
 			(at 7.62 0 270)
-			(size 2.4 1.6)
+			(size 1.6 1.6)
 			(drill 0.8)
 			(layers "*.Cu" "*.Mask")
@@
 		(target_delay_min 0)
 		(target_length 64)
-		(target_length_max 64.1)
+		(target_length_max 64.099999)
 		(target_length_min 63.9)
 		(target_skew 0)
@@
 		(last_status "tuned")
 		(last_track_width 0.2)
-		(last_tuning_length 64.000008)
+		(last_tuning_length 64.000007)
 		(max_amplitude 0.6)
 		(min_amplitude 0.2)
@@
 		(target_delay_min 0)
 		(target_length 64)
-		(target_length_max 64.1)
+		(target_length_max 64.099999)
 		(target_length_min 63.9)
 		(target_skew 0)

Commit message: Updated PCB Schematics
Added correct capacitor values and one missing resistor on USB card
Parts:
- C3, C4, C5, C6, C7, C8, C9: value 0.47uF -> 0.1uF
- U5: footprint Package_DIP:DIP-16_W7.62mm -> Package_DIP:DIP-16_W7.62mm_LongPads
Changed lines of the file:
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@@
 		)
 	)
-	(footprint "Package_DIP:DIP-16_W7.62mm"
+	(footprint "Package_DIP:DIP-16_W7.62mm_LongPads"
 		(layer "F.Cu")
 		(at 190.627 70.95 -90)
-		(descr "16-lead though-hole mounted DIP package, row spacing 7.62mm (300 mils)")
-		(tags "THT DIP DIL PDIP 2.54mm 7.62mm 300mil")
+		(descr "16-lead though-hole mounted DIP package, row spacing 7.62mm (300 mils), LongPads")
+		(tags "THT DIP DIL PDIP 2.54mm 7.62mm 300mil LongPads")
 		(property "Reference" "U5"
 			(at 3.81 -2.33 90)
@@
 		(duplicate_pad_numbers_are_jumpers no)
 		(fp_line
-			(start 1.16 19.11)
-			(end 6.46 19.11)
+			(start 1.56 19.11)
+			(end 6.06 19.11)
 			(stroke
 				(width 0.12)
@@
 		)
 		(fp_line
-			(start 6.46 19.11)
-			(end 6.46 -1.33)
+			(start 6.06 19.11)
+			(end 6.06 -1.33)
 			(stroke
 				(width 0.12)
@@
 		)
 		(fp_line
-			(start 1.16 -1.33)
-			(end 1.16 19.11)
+			(start 1.56 -1.33)
+			(end 1.56 19.11)
 			(stroke
 				(width 0.12)
@@
 		(fp_line
 			(start 2.81 -1.33)
-			(end 1.16 -1.33)
+			(end 1.56 -1.33)
 			(stroke
 				(width 0.12)
@@
 		)
 		(fp_line
-			(start 6.46 -1.33)
+			(start 6.06 -1.33)
 			(end 4.81 -1.33)
 			(stroke
@@
 		)
 		(fp_rect
-			(start -1.06 -1.52)
-			(end 8.67 19.3)
+			(start -1.45 -1.52)
+			(end 9.07 19.3)
 			(stroke
 				(width 0.05)
@@
 		(pad "1" thru_hole roundrect
 			(at 0 0 270)
-			(size 1.6 1.6)
+			(size 2.4 1.6)
 			(drill 0.8)
 			(layers "*.Cu" "*.Mask")
@@
 			(pintype "input")
 		)
-		(pad "2" thru_hole circle
+		(pad "2" thru_hole oval
 			(at 0 2.54 270)
-			(size 1.6 1.6)
+			(size 2.4 1.6)
 			(drill 0.8)
 			(layers "*.Cu" "*.Mask")
@@
 			(pintype "input")
 		)
-		(pad "3" thru_hole circle
+		(pad "3" thru_hole oval
 			(at 0 5.08 270)
-			(size 1.6 1.6)
+			(size 2.4 1.6)
 			(drill 0.8)
 			(layers "*.Cu" "*.Mask")
@@
 			(pintype "input")
 		)
-		(pad "4" thru_hole circle
+		(pad "4" thru_hole oval
 			(at 0 7.62 270)
-			(size 1.6 1.6)
+			(size 2.4 1.6)
 			(drill 0.8)
 			(layers "*.Cu" "*.Mask")
@@
 			(pintype "input")
 		)
-		(pad "5" thru_hole circle
+		(pad "5" thru_hole oval
 			(at 0 10.16 270)
-			(size 1.6 1.6)
+			(size 2.4 1.6)
 			(drill 0.8)
 			(layers "*.Cu" "*.Mask")
@@
 			(pintype "input")
 		)
-		(pad "6" thru_hole circle
+		(pad "6" thru_hole oval
 			(at 0 12.7 270)
-			(size 1.6 1.6)
+			(size 2.4 1.6)
 			(drill 0.8)
 			(layers "*.Cu" "*.Mask")
@@
 			(pintype "input")
 		)
-		(pad "7" thru_hole circle
+		(pad "7" thru_hole oval
 			(at 0 15.24 270)
-			(size 1.6 1.6)
+			(size 2.4 1.6)
 			(drill 0.8)
 			(layers "*.Cu" "*.Mask")
@@
 			(pintype "input")
 		)
-		(pad "8" thru_hole circle
+		(pad "8" thru_hole oval
 			(at 0 17.78 270)
-			(size 1.6 1.6)
+			(size 2.4 1.6)
 			(drill 0.8)
 			(layers "*.Cu" "*.Mask")
@@
 			(pintype "input")
 		)
-		(pad "9" thru_hole circle
+		(pad "9" thru_hole oval
 			(at 7.62 17.78 270)
-			(size 1.6 1.6)
+			(size 2.4 1.6)
 			(drill 0.8)
 			(layers "*.Cu" "*.Mask")
@@
 			(pintype "power_in")
 		)
-		(pad "10" thru_hole circle
+		(pad "10" thru_hole oval
 			(at 7.62 15.24 270)
-			(size 1.6 1.6)
+			(size 2.4 1.6)
 			(drill 0.8)
 			(layers "*.Cu" "*.Mask")
@@
 			(pintype "input")
 		)
-		(pad "11" thru_hole circle
+		(pad "11" thru_hole oval
 			(at 7.62 12.7 270)
-			(size 1.6 1.6)
+			(size 2.4 1.6)
 			(drill 0.8)
 			(layers "*.Cu" "*.Mask")
@@
 			(pintype "input")
 		)
-		(pad "12" thru_hole circle
+		(pad "12" thru_hole oval
 			(at 7.62 10.16 270)
-			(size 1.6 1.6)
+			(size 2.4 1.6)
 			(drill 0.8)
 			(layers "*.Cu" "*.Mask")
@@
 			(pintype "output")
 		)
-		(pad "13" thru_hole circle
+		(pad "13" thru_hole oval
 			(at 7.62 7.62 270)
-			(size 1.6 1.6)
+			(size 2.4 1.6)
 			(drill 0.8)
 			(layers "*.Cu" "*.Mask")
@@
 			(pintype "input")
 		)
-		(pad "14" thru_hole circle
+		(pad "14" thru_hole oval
 			(at 7.62 5.08 270)
-			(size 1.6 1.6)
+			(size 2.4 1.6)
 			(drill 0.8)
 			(layers "*.Cu" "*.Mask")
@@
 			(pintype "power_in")
 		)
-		(pad "15" thru_hole circle
+		(pad "15" thru_hole oval
 			(at 7.62 2.54 270)
-			(size 1.6 1.6)
+			(size 2.4 1.6)
 			(drill 0.8)
 			(layers "*.Cu" "*.Mask")
@@
 			(pintype "power_in")
 		)
-		(pad "16" thru_hole circle
+		(pad "16" thru_hole oval
 			(at 7.62 0 270)
-			(size 1.6 1.6)
+			(size 2.4 1.6)
 			(drill 0.8)
 			(layers "*.Cu" "*.Mask")
@@
 			)
 		)
-		(property "Value" "0.47uF"
+		(property "Value" "0.1uF"
 			(at 0 -3.12 0)
 			(layer "B.Fab")
@@
 			)
 		)
-		(property "Value" "0.47uF"
+		(property "Value" "0.1uF"
 			(at 0 -1.85 0)
 			(layer "B.Fab")
@@
 			)
 		)
-		(property "Value" "0.47uF"
+		(property "Value" "0.1uF"
 			(at 0 -1.85 0)
 			(layer "B.Fab")
@@
 			)
 		)
-		(property "Value" "0.47uF"
+		(property "Value" "0.1uF"
 			(at 0 -1.85 0)
 			(layer "B.Fab")
@@
 			)
 		)
-		(property "Value" "0.47uF"
+		(property "Value" "0.1uF"
 			(at 0 -1.85 0)
 			(layer "B.Fab")
@@
 			)
 		)
-		(property "Value" "0.47uF"
+		(property "Value" "0.1uF"
 			(at 5.1185 0 0)
 			(layer "B.Fab")
@@
 			)
 		)
-		(property "Value" "0.47uF"
+		(property "Value" "0.1uF"
 			(at 0 -1.85 0)
 			(layer "B.Fab")
