File: Loaf/PCB/PLC_Input_Slice/BREAD_slice_v2.kicad_sch (KiCad schematic)
At the start: 41 parts, among them J1 10018783-10200TLF, J2 Barrel_Jack, J3 DB25_Socket, U1 MCP4922-EP, U2 MCP4922-EP, U3 MCP4922-EP, U4 MCP4922-EP, U5 MCP3208, U6 MCP2561-E-P, U7 MCP2515-xSO, Y1 16MHZ Crystal

Commit message: Work on new new new new IO Slice
Parts:
- removed R3, R4: 10K, R_Axial_DIN0207_L6.3mm_D2.5mm_P10.16mm_Horizontal, symbol Device:R_US
- renumbered U4 to U1, U3 to U2, U2 to U3, U1 to U4
Connections:
- net +5V: no longer RN3.1 (common)
- net AIO0: now also U3.14 (VoutA); no longer U4.10 (VoutB)
- net AIO1: now also U3.10 (VoutB); no longer U4.14 (VoutA)
- net AIO2: now also U4.14 (VoutA); no longer U3.10 (VoutB)
- net AIO3: now also U4.10 (VoutB); no longer U3.14 (VoutA)
- net AIO4: now also U1.14 (VoutA); no longer U2.10 (VoutB)
- net AIO5: now also U1.10 (VoutB); no longer U2.14 (VoutA)
- net AIO6: now also U2.14 (VoutA); no longer U1.10 (VoutB)
- net AIO7: now also U2.10 (VoutB); no longer U1.14 (VoutA)
- net CAN_CS: now also RN3.7 (R6); no longer RN3.5 (R4)
- net DAC1: now also A1.15 (GPIO11), RN3.9 (R8), U1.3 (~{CS}); no longer A1.11 (GPIO8), RN3.7 (R6), U4.3 (~{CS})
- net DAC2: now also A1.14 (GPIO10), RN3.8 (R7), U2.3 (~{CS}); no longer A1.12 (GPIO9), RN3.6 (R5), U3.3 (~{CS})
- net DAC3: now also A1.12 (GPIO9), RN3.6 (R5), U3.3 (~{CS}); no longer A1.14 (GPIO10), RN3.8 (R7), U2.3 (~{CS})
- net DAC4: now also A1.11 (GPIO8), RN3.5 (R4), U4.3 (~{CS}); no longer A1.15 (GPIO11), RN3.9 (R8), U1.3 (~{CS})
- net ESTOP: now also A1.7 (GPIO5), RN3.2 (R1); no longer A1.9 (GPIO6)
- net GND: now also RN3.1 (common)
- net SHDN: now also A1.9 (GPIO6), RN3.3 (R2); no longer A1.7 (GPIO5)

Commit message: I/O Slice Updated
Connections:
- net AIO0: now also RN2.2 (R1); no longer RN2.9 (R8)
- net AIO1: now also RN2.3 (R2); no longer RN2.8 (R7)
- net AIO2: now also RN2.4 (R3); no longer RN2.7 (R6)
- net AIO3: now also RN2.5 (R4); no longer RN2.6 (R5)
- net AIO4: now also RN2.6 (R5); no longer RN2.5 (R4)
- net AIO5: now also RN2.7 (R6); no longer RN2.4 (R3)
- net AIO6: now also RN2.8 (R7); no longer RN2.3 (R2)
- net AIO7: now also RN2.9 (R8); no longer RN2.2 (R1)
- net DIO0: now also RN1.2 (R1); no longer RN1.9 (R8)
- net DIO1: now also RN1.3 (R2); no longer RN1.8 (R7)
- net DIO2: now also RN1.4 (R3); no longer RN1.7 (R6)
- net DIO3: now also RN1.5 (R4); no longer RN1.6 (R5)
- net DIO4: now also RN1.6 (R5); no longer RN1.5 (R4)
- net DIO5: now also RN1.7 (R6); no longer RN1.4 (R3)
- net DIO6: now also RN1.8 (R7); no longer RN1.3 (R2)
- net DIO7: now also RN1.9 (R8); no longer RN1.2 (R1)
- net Sl1Lt: now also A1.20 (GPIO15)
- net URX: now also J3.5; no longer J3.18 (P18)
- net UTX: now also J3.18 (P18); no longer J3.5
Changed lines of the file:
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@@
 	(wire
 		(pts
+			(xy 31.75 88.9) (xy 36.83 88.9)
+		)
+		(stroke
+			(width 0)
+			(type default)
+		)
+	)
+	(wire
+		(pts
 			(xy 166.37 106.68) (xy 161.29 106.68)
 		)
@@
 	(wire
 		(pts
-			(xy 130.81 146.05) (xy 135.89 146.05)
+			(xy 130.81 158.75) (xy 135.89 158.75)
 		)
 		(stroke
@@
 	(wire
 		(pts
-			(xy 130.81 153.67) (xy 135.89 153.67)
+			(xy 130.81 151.13) (xy 135.89 151.13)
 		)
 		(stroke
@@
 	(wire
 		(pts
-			(xy 130.81 148.59) (xy 135.89 148.59)
+			(xy 130.81 156.21) (xy 135.89 156.21)
 		)
 		(stroke
@@
 	(wire
 		(pts
-			(xy 130.81 151.13) (xy 135.89 151.13)
+			(xy 130.81 153.67) (xy 135.89 153.67)
 		)
 		(stroke
@@
 	(wire
 		(pts
-			(xy 130.81 161.29) (xy 135.89 161.29)
+			(xy 130.81 143.51) (xy 135.89 143.51)
 		)
 		(stroke
@@
 	(wire
 		(pts
-			(xy 130.81 156.21) (xy 135.89 156.21)
+			(xy 130.81 148.59) (xy 135.89 148.59)
 		)
 		(stroke
@@
 	(wire
 		(pts
-			(xy 130.81 158.75) (xy 135.89 158.75)
+			(xy 130.81 146.05) (xy 135.89 146.05)
 		)
 		(stroke
@@
 	(wire
 		(pts
-			(xy 130.81 143.51) (xy 135.89 143.51)
+			(xy 130.81 161.29) (xy 135.89 161.29)
 		)
 		(stroke
@@
 	)
 	(label "UTX"
-		(at 128.27 189.23 90)
+		(at 130.81 189.23 90)
 		(effects
 			(font
@@
 	)
 	(label "DIO0"
-		(at 151.13 161.29 0)
+		(at 151.13 143.51 0)
 		(effects
 			(font
@@
 	)
 	(label "DIO1"
-		(at 151.13 158.75 0)
+		(at 151.13 146.05 0)
 		(effects
 			(font
@@
 	)
 	(label "URX"
-		(at 130.81 189.23 90)
+		(at 128.27 189.23 90)
 		(effects
 			(font
@@
 	)
 	(label "DIO3"
-		(at 151.13 153.67 0)
+		(at 151.13 151.13 0)
 		(effects
 			(font
@@
 	)
 	(label "AIO2"
-		(at 130.81 156.21 0)
+		(at 130.81 148.59 0)
 		(effects
 			(font
@@
 	)
 	(label "AIO1"
-		(at 130.81 158.75 0)
+		(at 130.81 146.05 0)
 		(effects
 			(font
@@
 	)
 	(label "AIO7"
-		(at 130.81 143.51 0)
+		(at 130.81 161.29 0)
 		(effects
 			(font
@@
 	)
 	(label "AIO5"
-		(at 130.81 148.59 0)
+		(at 130.81 156.21 0)
 		(effects
 			(font
@@
 	)
 	(label "AIO6"
-		(at 130.81 146.05 0)
+		(at 130.81 158.75 0)
 		(effects
 			(font
@@
 	)
 	(label "AIO3"
-		(at 130.81 153.67 0)
+		(at 130.81 151.13 0)
 		(effects
 			(font
@@
 	)
 	(label "DIO7"
-		(at 151.13 143.51 0)
+		(at 151.13 161.29 0)
 		(effects
 			(font
@@
 	)
 	(label "DIO4"
-		(at 151.13 151.13 0)
+		(at 151.13 153.67 0)
 		(effects
 			(font
@@
 	)
 	(label "AIO4"
-		(at 130.81 151.13 0)
+		(at 130.81 153.67 0)
 		(effects
 			(font
@@
 		)
 	)
+	(label "Sl1Lt"
+		(at 31.75 88.9 0)
+		(effects
+			(font
+				(size 1.27 1.27)
+			)
+			(justify left bottom)
+		)
+	)
 	(label "CANRX"
 		(at 236.22 144.78 0)
@@
 	)
 	(label "DIO6"
-		(at 151.13 146.05 0)
+		(at 151.13 158.75 0)
 		(effects
 			(font
@@
 	)
 	(label "DIO5"
-		(at 151.13 148.59 0)
+		(at 151.13 156.21 0)
 		(effects
 			(font
@@
 	)
 	(label "AIO0"
-		(at 130.81 161.29 0)
+		(at 130.81 143.51 0)
 		(effects
 			(font
@@
 	)
 	(label "DIO2"
-		(at 151.13 156.21 0)
+		(at 151.13 148.59 0)
 		(effects
 			(font

Commit message: Slight updates
Parts:
- C10, C11, C12, C14, C15, C16: value 10pF -> 150pF
Changed lines of the file:
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@@
 			)
 		)
-		(property "Value" "10pF"
+		(property "Value" "150pF"
 			(at 139.7 110.236 90)
 			(hide yes)
@@
 			)
 		)
-		(property "Value" "10pF"
+		(property "Value" "150pF"
 			(at 139.7 117.856 90)
 			(hide yes)
@@
 			)
 		)
-		(property "Value" "10pF"
+		(property "Value" "150pF"
 			(at 157.48 110.236 90)
 			(hide yes)
@@
 			)
 		)
-		(property "Value" "10pF"
+		(property "Value" "150pF"
 			(at 139.7 125.476 90)
 			(hide yes)
@@
 			)
 		)
-		(property "Value" "10pF"
+		(property "Value" "150pF"
 			(at 157.48 125.476 90)
 			(hide yes)
@@
 			)
 		)
-		(property "Value" "10pF"
+		(property "Value" "150pF"
 			(at 157.48 117.856 90)
 			(hide yes)

Commit message: Redid io gerbers
Parts:
- added F1: Polyfuse, Fuse_2920_7451Metric_Pad2.10x5.45mm_HandSolder, symbol Device:Polyfuse
Connections:
- net +12V: now also F1.1; no longer J2.1
- new net 12VO: F1.2, J2.1
Changed lines of the file:
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@@
 	)
 	(symbol
+		(lib_id "power:+12V")
+		(at 113.03 113.03 90)
+		(unit 1)
+		(body_style 1)
+		(exclude_from_sim no)
+		(in_bom yes)
+		(on_board yes)
+		(in_pos_files yes)
+		(dnp no)
+		(fields_autoplaced yes)
+		(property "Reference" "#PWR064"
+			(at 116.84 113.03 0)
+			(hide yes)
+			(show_name no)
+			(do_not_autoplace no)
+			(effects
+				(font
+					(size 1.27 1.27)
+				)
+			)
+		)
+		(property "Value" "+12V"
+			(at 109.22 113.0299 90)
+			(show_name no)
+			(do_not_autoplace no)
+			(effects
+				(font
+					(size 1.27 1.27)
+				)
+				(justify left)
+			)
+		)
+		(property "Footprint" ""
+			(at 113.03 113.03 0)
+			(hide yes)
+			(show_name no)
+			(do_not_autoplace no)
+			(effects
+				(font
+					(size 1.27 1.27)
+				)
+			)
+		)
+		(property "Datasheet" ""
+			(at 113.03 113.03 0)
+			(hide yes)
+			(show_name no)
+			(do_not_autoplace no)
+			(effects
+				(font
+					(size 1.27 1.27)
+				)
+			)
+		)
+		(property "Description" "Power symbol creates a global label with name \"+12V\""
+			(at 113.03 113.03 0)
+			(hide yes)
+			(show_name no)
+			(do_not_autoplace no)
+			(effects
+				(font
+					(size 1.27 1.27)
+				)
+			)
+		)
+		(pin "1"
+		)
+		(instances
+			(project "BREAD_slice_v2"
+				(path "/7f913798-a7fb-4519-b930-d05e163d3032"
+					(reference "#PWR064")
+					(unit 1)
+				)
+			)
+		)
+	)
+	(symbol
 		(lib_id "Connector:Barrel_Jack")
 		(at 111.76 129.54 0)
@@
 	)
 	(symbol
-		(lib_id "power:GND")
-		(at 270.51 124.46 0)
-		(mirror x)
+		(lib_id "Device:Polyfuse")
+		(at 116.84 113.03 90)
 		(unit 1)
 		(body_style 1)
@@
 		(in_pos_files yes)
 		(dnp no)
-		(property "Reference" "#PWR056"
-			(at 270.51 118.11 0)
-			(hide yes)
+		(fields_autoplaced yes)
+		(property "Reference" "F1"
+			(at 116.84 106.68 90)
 			(show_name no)
 			(do_not_autoplace no)
@@
 			)
 		)
-		(property "Value" "GND"
-			(at 266.7 124.46 0)
+		(property "Value" "Polyfuse"
+			(at 116.84 109.22 90)
 			(show_name no)
 			(do_not_autoplace no)
@@
 			)
 		)
-		(property "Footprint" ""
-			(at 270.51 124.46 0)
+		(property "Footprint" "Fuse_2920_7451Metric_Pad2.10x5.45mm_HandSolder"
+			(at 121.92 111.76 0)
 			(hide yes)
 			(show_name no)
@@
 					(size 1.27 1.27)
 				)
+				(justify left)
 			)
 		)
 		(property "Datasheet" ""
-			(at 270.51 124.46 0)
+			(at 116.84 113.03 0)
 			(hide yes)
 			(show_name no)
@@
 			)
 		)
-		(property "Description" ""
-			(at 270.51 124.46 0)
+		(property "Description" "Resettable fuse, polymeric positive temperature coefficient"
+			(at 116.84 113.03 0)
 			(hide yes)
 			(show_name no)
@@
 			)
 		)
+		(pin "2"
+		)
 		(pin "1"
 		)
@@
 			(project "BREAD_slice_v2"
 				(path "/7f913798-a7fb-4519-b930-d05e163d3032"
-					(reference "#PWR056")
+					(reference "F1")
 					(unit 1)
 				)
@@
 	)
 	(symbol
-		(lib_id "power:+12V")
-		(at 119.38 127 270)
+		(lib_id "power:GND")
+		(at 270.51 124.46 0)
+		(mirror x)
 		(unit 1)
 		(body_style 1)
@@
 		(in_pos_files yes)
 		(dnp no)
-		(fields_autoplaced yes)
-		(property "Reference" "#PWR062"
-			(at 115.57 127 0)
+		(property "Reference" "#PWR056"
+			(at 270.51 118.11 0)
 			(hide yes)
 			(show_name no)
@@
 			)
 		)
-		(property "Value" "+12V"
-			(at 123.19 127.0001 90)
+		(property "Value" "GND"
+			(at 266.7 124.46 0)
 			(show_name no)
 			(do_not_autoplace no)
@@
 					(size 1.27 1.27)
 				)
-				(justify left)
 			)
 		)
 		(property "Footprint" ""
-			(at 119.38 127 0)
+			(at 270.51 124.46 0)
 			(hide yes)
 			(show_name no)
@@
 		)
 		(property "Datasheet" ""
-			(at 119.38 127 0)
+			(at 270.51 124.46 0)
 			(hide yes)
 			(show_name no)
@@
 			)
 		)
-		(property "Description" "Power symbol creates a global label with name \"+12V\""
-			(at 119.38 127 0)
+		(property "Description" ""
+			(at 270.51 124.46 0)
 			(hide yes)
 			(show_name no)
@@
 			(project "BREAD_slice_v2"
 				(path "/7f913798-a7fb-4519-b930-d05e163d3032"
-					(reference "#PWR062")
+					(reference "#PWR056")
 					(unit 1)
 				)
@@
 	)
 	(symbol
+		(lib_id "power:+12V")
+		(at 119.38 127 270)
+		(unit 1)
+		(body_style 1)
+		(exclude_from_sim no)
+		(in_bom yes)
+		(on_board yes)
+		(in_pos_files yes)
+		(dnp no)
+		(fields_autoplaced yes)
+		(property "Reference" "#PWR066"
+			(at 115.57 127 0)
+			(hide yes)
+			(show_name no)
+			(do_not_autoplace no)
+			(effects
+				(font
+					(size 1.27 1.27)
+				)
+			)
+		)
+		(property "Value" "12VO"
+			(at 123.19 126.9999 90)
+			(show_name no)
+			(do_not_autoplace no)
+			(effects
+				(font
+					(size 1.27 1.27)
+				)
+				(justify left)
+			)
+		)
+		(property "Footprint" ""
+			(at 119.38 127 0)
+			(hide yes)
+			(show_name no)
+			(do_not_autoplace no)
+			(effects
+				(font
+					(size 1.27 1.27)
+				)
+			)
+		)
+		(property "Datasheet" ""
+			(at 119.38 127 0)
+			(hide yes)
+			(show_name no)
+			(do_not_autoplace no)
+			(effects
+				(font
+					(size 1.27 1.27)
+				)
+			)
+		)
+		(property "Description" "Power symbol creates a global label with name \"+12V\""
+			(at 119.38 127 0)
+			(hide yes)
+			(show_name no)
+			(do_not_autoplace no)
+			(effects
+				(font
+					(size 1.27 1.27)
+				)
+			)
+		)
+		(pin "1"
+		)
+		(instances
+			(project "BREAD_slice_v2"
+				(path "/7f913798-a7fb-4519-b930-d05e163d3032"
+					(reference "#PWR066")
+					(unit 1)
+				)
+			)
+		)
+	)
+	(symbol
 		(lib_id "Analog_DAC:MCP4922-EP")
 		(at 228.6 48.26 270)
@@
 					(unit 1)
 				)
+			)
+		)
+	)
+	(symbol
+		(lib_id "power:+12V")
+		(at 120.65 113.03 270)
+		(unit 1)
+		(body_style 1)
+		(exclude_from_sim no)
+		(in_bom yes)
+		(on_board yes)
+		(in_pos_files yes)
+		(dnp no)
+		(fields_autoplaced yes)
+		(property "Reference" "#PWR065"
+			(at 116.84 113.03 0)
+			(hide yes)
+			(show_name no)
+			(do_not_autoplace no)
+			(effects
+				(font
+					(size 1.27 1.27)
+				)
+			)
+		)
+		(property "Value" "12VO"
+			(at 124.46 113.0299 90)
+			(show_name no)
+			(do_not_autoplace no)
+			(effects
+				(font
+					(size 1.27 1.27)
+				)
+				(justify left)
+			)
+		)
+		(property "Footprint" ""
+			(at 120.65 113.03 0)
+			(hide yes)
+			(show_name no)
+			(do_not_autoplace no)
+			(effects
+				(font
+					(size 1.27 1.27)
+				)
+			)
+		)
+		(property "Datasheet" ""
+			(at 120.65 113.03 0)
+			(hide yes)
+			(show_name no)
+			(do_not_autoplace no)
+			(effects
+				(font
+					(size 1.27 1.27)
+				)
+			)
+		)
+		(property "Description" "Power symbol creates a global label with name \"+12V\""
+			(at 120.65 113.03 0)
+			(hide yes)
+			(show_name no)
+			(do_not_autoplace no)
+			(effects
+				(font
+					(size 1.27 1.27)
+				)
+			)
+		)
+		(pin "1"
+		)
+		(instances
+			(project "BREAD_slice_v2"
+				(path "/7f913798-a7fb-4519-b930-d05e163d3032"
+					(reference "#PWR065")
+					(unit 1)
+				)
