File: Loaf/PCB/VRM Module/VRM Module.kicad_sch (KiCad schematic)
At the start: 12 parts, among them U1 TPS564242DRLR

Commit message: IO PCB redesign progress upload
Switching to pi pico for better performance and to keep UART interface
Parts:
- removed C1: 10uF, C_1206_3216Metric_Pad1.33x1.80mm_HandSolder, symbol Device:C
- removed U1: TPS564242DRLR, SOT-563, symbol 2026-10-14_17-23-55:TPS564242DRLR
- added C1: 10uF, CP_Radial_D5.0mm_P2.50mm, symbol Device:C_Polarized_US
- added C6: 22uF, CP_Radial_D5.0mm_P2.50mm, symbol Device:C_Polarized_US
- added H1: MountingHole_Pad, MountingHole:MountingHole_3.2mm_M3_DIN965_Pad, symbol Mechanical:MountingHole_Pad
- added U1: TPS54429PWP, Texas_HTSSOP-14-1EP_4.4x5mm_P0.65mm_EP3.4x5mm_Mask2.94x3.34mm, symbol 2026-10-15_20-36-02:TPS54429PWP
- C2: value 100nF -> 1uF
- C3: value 33pF -> 3.3uF
- C4: value 22uF -> 100nF
- C5: value 100nF -> 10pF
- J1: renamed from VRM1; value VRM -> VRM Pin Header
- L1: value 1.8uH -> 3.3uH; footprint (none) -> R_1206_3216Metric_Pad1.30x1.75mm_HandSolder
- R1: value 100k -> 10k; footprint (none) -> R_1206_3216Metric_Pad1.30x1.75mm_HandSolder
- R2: value 15.8k -> 105k; footprint (none) -> R_1206_3216Metric_Pad1.30x1.75mm_HandSolder
- R3: value 220k -> 133k; footprint (none) -> R_1206_3216Metric_Pad1.30x1.75mm_HandSolder
- R4: value 30k -> 24k; footprint (none) -> R_1206_3216Metric_Pad1.30x1.75mm_HandSolder
Connections:
- net +12V: now also R1.1, C1.1, U1.13 (VIN1), U1.14 (VIN2); no longer C2.1, R1.2
- net +5V: now also C5.2, L1.2, C6.1, U1.1 (VO); no longer C3.1, C4.1, C5.1, L1.1
- net GND: now also C2.1, C3.1, C1.2, C6.2, H1.1, U1.15 (EPAD), U1.5 (GND), U1.8 (PGND1), U1.9 (PGND2); no longer C2.2, C4.2, C5.2, R2.1
- net EN: no longer names the net of R2.2
- net EN: now also U1.6 (PG); no longer R1.1
- net FB renamed VFB
- net VFB: now also C5.1, U1.2 (VFB); no longer C3.2
- new net: C4.2, L1.1, U1.10 (SW1), U1.11 (SW2)
- new net: C3.2, U1.4 (SS)
- new net: C4.1, U1.12 (VBST)
- new net: R1.2, U1.7 (EN)
- new net VREG: C2.2, R2.1, U1.3 (VREG5)
