File: Loaf/PCB/5V4A VRM Module/VRM Module.kicad_pcb (KiCad board)
At the start: 2 copper layers, 37 x 21.5 mm, 14 parts, among them J1 VRM Pin Header, U1 TPS54429PWP

Commit message: Added OSHE branding to VRM
Parts:
- added Logo1: Logo_Open_Hardware_Small, Symbol:OSHW-Symbol_6.7x6mm_SilkScreen, F.Cu at (139.1, 77.7)
- C1, C6: moved to F.Cu
- moved C6 0.38 mm to (150.8, 79.4)
Routing:
- net GND: vias 1 -> 29
Other:
- board text added: "BREAD I/O Board 5V4A VRM V1"
- board text added: "oshe.io Rev. 2026"

Commit message: Peter recommended PCB changes
Connections:
- J1 pad 1: +3.3V -> Net-(J1-Pin_1)
- J1 pad 15: +3.3V -> Net-(J1-Pin_15)
- J1 pad 16: +3.3V -> Net-(J1-Pin_15)
- J1 pad 2: +3.3V -> Net-(J1-Pin_1)
Routing:
- net +3.3V: track 10.2 -> 0.00 mm
- net Net-(J1-Pin_15): track 0.00 -> 5.08 mm
- net Net-(J1-Pin_1): track 0.00 -> 5.08 mm
- net +12V: track 47.2 -> 47.9 mm
Changed lines of the file:
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@@
 			(layers "*.Cu" "*.Mask")
 			(remove_unused_layers no)
-			(net "+3.3V")
+			(net "Net-(J1-Pin_1)")
 			(pinfunction "Pin_1_1")
 			(pintype "passive")
@@
 			(layers "*.Cu" "*.Mask")
 			(remove_unused_layers no)
-			(net "+3.3V")
+			(net "Net-(J1-Pin_1)")
 			(pinfunction "Pin_2_2")
 			(pintype "passive")
@@
 			(layers "*.Cu" "*.Mask")
 			(remove_unused_layers no)
-			(net "+3.3V")
+			(net "Net-(J1-Pin_15)")
 			(pinfunction "Pin_15_15")
 			(pintype "passive")
@@
 			(layers "*.Cu" "*.Mask")
 			(remove_unused_layers no)
-			(net "+3.3V")
+			(net "Net-(J1-Pin_15)")
 			(pinfunction "Pin_16_16")
 			(pintype "passive")
@@
 	)
 	(segment
-		(start 146.25 83.7022)
+		(start 147.066 84.5182)
+		(end 146.25 84.5182)
+		(width 0.2)
+		(layer "F.Cu")
+		(net "/VREG")
+	)
+	(segment
+		(start 146.25 84.5182)
 		(end 146.25 82.75)
 		(width 0.2)
@@
 	(segment
 		(start 147.066 84.5182)
-		(end 146.25 83.7022)
-		(width 0.2)
-		(layer "F.Cu")
-		(net "/VREG")
-	)
-	(segment
-		(start 147.066 84.5182)
 		(end 146.2318 84.5182)
 		(width 0.2)
@@
 	)
 	(segment
+		(start 168.004996 78.84)
+		(end 170.544996 78.84)
+		(width 2)
+		(layer "F.Cu")
+		(net "+5V")
+	)
+	(segment
+		(start 165.862 91.54)
+		(end 168 91.54)
+		(width 0.2)
+		(layer "F.Cu")
+		(net "+5V")
+	)
+	(segment
 		(start 168 78.84)
 		(end 167.433726 78.84)
@@
 	)
 	(segment
-		(start 168.004996 78.84)
-		(end 170.544996 78.84)
-		(width 2)
-		(layer "F.Cu")
-		(net "+5V")
-	)
-	(segment
-		(start 143.604 94.45)
-		(end 163.53 94.45)
-		(width 2)
-		(layer "F.Cu")
-		(net "+5V")
-	)
-	(segment
-		(start 150.85 81.25)
-		(end 150.85 79)
+		(start 145.538 75.95)
+		(end 143.604 77.884)
+		(width 2)
+		(layer "F.Cu")
+		(net "+5V")
+	)
+	(segment
+		(start 163.53 94.45)
+		(end 166.44 91.54)
+		(width 2)
+		(layer "F.Cu")
+		(net "+5V")
+	)
+	(segment
+		(start 161.66 91.54)
+		(end 161.6 91.6)
+		(width 0.2)
+		(layer "F.Cu")
+		(net "+5V")
+	)
+	(segment
+		(start 150.85 82.6925)
+		(end 150.85 75.95)
 		(width 1.5)
+		(layer "F.Cu")
+		(net "+5V")
+	)
+	(segment
+		(start 167.433726 78.84)
+		(end 164.543726 75.95)
+		(width 2)
+		(layer "F.Cu")
+		(net "+5V")
+	)
+	(segment
+		(start 143.604 92.55)
+		(end 145.504 94.45)
+		(width 2)
 		(layer "F.Cu")
 		(net "+5V")
@@
 	)
 	(segment
-		(start 164.475 91.54)
-		(end 164.435 91.5)
-		(width 0.2)
-		(layer "F.Cu")
-		(net "+5V")
-	)
-	(segment
-		(start 164.543726 75.95)
-		(end 143.604 75.95)
-		(width 2)
-		(layer "F.Cu")
-		(net "+5V")
-	)
-	(segment
-		(start 150.85 82.6925)
-		(end 150.8725 82.715)
-		(width 1.5)
-		(layer "F.Cu")
-		(net "+5V")
-	)
-	(segment
-		(start 150.85 81.25)
+		(start 150.8725 82.715)
 		(end 150.85 82.6925)
 		(width 1.5)
@@
 	)
 	(segment
-		(start 161.7 91.5)
-		(end 161.6 91.6)
-		(width 0.2)
-		(layer "F.Cu")
-		(net "+5V")
-	)
-	(segment
-		(start 164.475 91.54)
-		(end 168 91.54)
-		(width 0.2)
+		(start 145.504 94.45)
+		(end 163.53 94.45)
+		(width 2)
+		(layer "F.Cu")
+		(net "+5V")
+	)
+	(segment
+		(start 143.604 77.884)
+		(end 143.604 92.55)
+		(width 2)
 		(layer "F.Cu")
 		(net "+5V")
@@
 	)
 	(segment
-		(start 164.435 91.5)
-		(end 161.7 91.5)
-		(width 0.2)
-		(layer "F.Cu")
-		(net "+5V")
-	)
-	(segment
-		(start 167.433726 78.84)
-		(end 164.543726 75.95)
-		(width 2)
-		(layer "F.Cu")
-		(net "+5V")
-	)
-	(segment
-		(start 150.85 79)
+		(start 164.543726 75.95)
+		(end 145.538 75.95)
+		(width 2)
+		(layer "F.Cu")
+		(net "+5V")
+	)
+	(segment
+		(start 165.862 91.54)
+		(end 161.66 91.54)
+		(width 0.2)
+		(layer "F.Cu")
+		(net "+5V")
+	)
+	(segment
+		(start 150.85 75.95)
 		(end 147.8 75.95)
 		(width 1.5)
@@
 		(net "+5V")
 	)
-	(segment
-		(start 163.53 94.45)
-		(end 166.44 91.54)
-		(width 2)
-		(layer "F.Cu")
-		(net "+5V")
-	)
-	(segment
-		(start 143.604 75.95)
-		(end 143.604 94.45)
-		(width 2)
-		(layer "F.Cu")
-		(net "+5V")
-	)
-	(via
-		(at 164.475 91.54)
-		(size 0.7064)
-		(drill 0.3)
-		(layers "F.Cu" "B.Cu")
+	(via
+		(at 165.862 91.54)
+		(size 0.7064)
+		(drill 0.3)
+		(layers "F.Cu" "B.Cu")
+		(net "+5V")
+	)
+	(segment
+		(start 165.862 91.54)
+		(end 164.475 90.153)
+		(width 0.2)
+		(layer "B.Cu")
+		(net "+5V")
+	)
+	(segment
+		(start 164.475 87.2)
+		(end 163.3 86.025)
+		(width 0.2)
+		(layer "B.Cu")
 		(net "+5V")
 	)
@@
 	)
 	(segment
-		(start 163.3 86.025)
-		(end 164.475 87.2)
-		(width 0.2)
-		(layer "B.Cu")
-		(net "+5V")
-	)
-	(segment
 		(start 170.54 91.54)
 		(end 168 91.54)
@@
 	)
 	(segment
-		(start 164.475 87.2)
-		(end 164.475 91.54)
+		(start 164.475 90.153)
+		(end 164.475 87.2)
 		(width 0.2)
 		(layer "B.Cu")
@@
 	)
 	(segment
-		(start 159.3 84.85)
-		(end 160.6 83.55)
-		(width 0.2)
-		(layer "F.Cu")
-		(net "+12V")
-	)
-	(segment
 		(start 167.63 83.55)
 		(end 168 83.92)
@@
 	)
 	(segment
-		(start 157.9 89.1)
-		(end 159.3 87.7)
-		(width 0.2)
-		(layer "F.Cu")
-		(net "+12V")
-	)
-	(segment
 		(start 168.004996 86.46)
 		(end 170.544996 86.46)
@@
 	)
 	(segment
+		(start 159.3 83.55)
+		(end 160.6 83.55)
+		(width 0.2)
+		(layer "F.Cu")
+		(net "+12V")
+	)
+	(segment
+		(start 159.3 87.7)
+		(end 159.3 83.55)
+		(width 0.2)
+		(layer "F.Cu")
+		(net "+12V")
+	)
+	(segment
+		(start 156.6 89.1)
+		(end 157.9 89.1)
+		(width 0.2)
+		(layer "F.Cu")
+		(net "+12V")
+	)
+	(segment
 		(start 170.544996 83.92)
 		(end 168.004996 83.92)
@@
 		(end 168.004996 83.92)
 		(width 2)
-		(layer "F.Cu")
-		(net "+12V")
-	)
-	(segment
-		(start 159.3 87.7)
-		(end 159.3 84.85)
-		(width 0.2)
-		(layer "F.Cu")
-		(net "+12V")
-	)
-	(segment
-		(start 156.6 89.1)
-		(end 157.9 89.1)
-		(width 0.2)
 		(layer "F.Cu")
 		(net "+12V")
@@
 	)
 	(segment
+		(start 157.9 89.1)
+		(end 159.3 87.7)
+		(width 0.2)
+		(layer "F.Cu")
+		(net "+12V")
+	)
+	(segment
 		(start 168 86.46)
 		(end 168 83.92)
@@
 		(width 2)
 		(layer "F.Cu")
-		(net "+3.3V")
+		(net "Net-(J1-Pin_1)")
+	)
+	(segment
+		(start 170.54 94.08)
+		(end 168 94.08)
+		(width 2)
+		(layer "B.Cu")
+		(net "Net-(J1-Pin_1)")
 	)
 	(segment
@@
 		(width 2)
 		(layer "F.Cu")
-		(net "+3.3V")
-	)
-	(segment
-		(start 170.54 94.08)
-		(end 168 94.08)
-		(width 2)
-		(layer "B.Cu")
-		(net "+3.3V")
+		(net "Net-(J1-Pin_15)")
 	)
 	(segment
@@
 		(width 2)
 		(layer "B.Cu")
-		(net "+3.3V")
+		(net "Net-(J1-Pin_15)")
 	)
 	(zone
