File: Loaf/PCB/5V4A VRM Module/VRM Module.kicad_sch (KiCad schematic)
At the start: 14 parts, among them J1 VRM Pin Header, U1 TPS54429PWP

Commit message: Peter recommended PCB changes
Connections:
- net +3.3V: no longer names the net of J1.1 (Pin_1), J1.2 (Pin_2)
- net +3.3V: no longer J1.15 (Pin_15), J1.16 (Pin_16)
- new net: J1.15 (Pin_15), J1.16 (Pin_16)
